File: pcb/radtel.kicad_pcb (KiCad board)
At the start: 2 copper layers, 50 x 23.2 mm, 53 parts, among them IC1 ADP3335, IC2 Si4460, IC3 STM32F072CBT6, M3_MOUNT VAL**, P1 PWR, P2 UART, P3 USB_OTG, P4 SWD, P5 ANTENNA, Y1 26MHz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

Commit message: move some capacitors a bit
Parts:
- moved C13 3.16 mm to (108.5, 107.5)
- moved C10 2.29 mm to (111.1, 107.5)
Routing:
- net GND: track 51.1 -> 53.7 mm
- net +3V3: track 85.4 -> 84.5 mm
Changed lines of the file:
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@@
-(kicad_pcb (version 4) (host pcbnew 0.201508100901+6080~28~ubuntu14.04.1-product)
+(kicad_pcb (version 4) (host pcbnew 0.201511061201+6302~30~ubuntu14.04.1-product)
   (general
     (links 124)
     (no_connects 0)
-    (area 78.525 86.875 148.027381 117.405952)
+    (area 78.525 88.375 133.536905 117.405952)
     (thickness 1.6)
     (drawings 16)
-    (tracks 395)
+    (tracks 401)
     (zones 0)
     (modules 53)
@@
   )
   (module radtel:C0603 (layer F.Cu)
-    (at 111.5 109.75)
+    (at 111.1 107.5)
     (fp_text reference C10 (at 0.7 -1.35) (layer F.SilkS) hide
       (effects (font (size 1 1) (thickness 0.15)))
@@
   )
   (module radtel:C0603 (layer F.Cu)
-    (at 111.5 108.5)
+    (at 108.5 107.5)
     (fp_text reference C13 (at 0.7 -1.35) (layer F.SilkS) hide
       (effects (font (size 1 1) (thickness 0.15)))
@@
   (segment (start 89.75 109.25) (end 91.25 109.25) (width 0.25) (layer F.Cu) (net 1))
   (segment (start 91.25 109.25) (end 91.5 109.5) (width 0.25) (layer F.Cu) (net 1))
+  (via (at 112.5 108.25) (size 0.6) (drill 0.4) (layers F.Cu B.Cu) (net 2))
+  (segment (start 112.5 107.5) (end 112.5 108.25) (width 0.25) (layer F.Cu) (net 2))
+  (segment (start 109.9 107.5) (end 109.9 106.85) (width 0.25) (layer F.Cu) (net 2))
+  (segment (start 109.9 106.85) (end 110 106.75) (width 0.25) (layer F.Cu) (net 2))
+  (segment (start 110 106.75) (end 112.4 106.75) (width 0.25) (layer F.Cu) (net 2))
+  (segment (start 112.4 106.75) (end 112.5 106.85) (width 0.25) (layer F.Cu) (net 2))
+  (segment (start 112.5 106.85) (end 112.5 107.5) (width 0.25) (layer F.Cu) (net 2))
   (segment (start 114.75 95.5) (end 115.25 95.5) (width 0.25) (layer F.Cu) (net 2))
   (via (at 115.25 95.5) (size 0.6) (drill 0.4) (layers F.Cu B.Cu) (net 2))
@@
   (segment (start 117.4 109.5) (end 118 109.5) (width 0.25) (layer F.Cu) (net 2))
   (segment (start 118 109.5) (end 118.6 109.5) (width 0.25) (layer F.Cu) (net 2))
-  (segment (start 112.9 109.75) (end 112.9 110.7) (width 0.25) (layer F.Cu) (net 2))
-  (via (at 112.9 110.7) (size 0.6) (drill 0.4) (layers F.Cu B.Cu) (net 2))
-  (segment (start 112.9 108.5) (end 112.9 109.75) (width 0.25) (layer F.Cu) (net 2))
   (via (at 107.2 112.5) (size 0.6) (drill 0.4) (layers F.Cu B.Cu) (net 2))
   (segment (start 106.65 112.5) (end 107.2 112.5) (width 0.25) (layer F.Cu) (net 2))
@@
   (segment (start 106.83 93.77) (end 108.37 93.77) (width 0.25) (layer F.Cu) (net 2))
   (segment (start 108.37 93.77) (end 108.5 93.9) (width 0.25) (layer F.Cu) (net 2))
+  (segment (start 110.825001 108.424999) (end 111.1 108.15) (width 0.25) (layer F.Cu) (net 3))
+  (segment (start 111.1 108.15) (end 111.1 107.5) (width 0.25) (layer F.Cu) (net 3))
+  (segment (start 108.774999 108.424999) (end 110.825001 108.424999) (width 0.25) (layer F.Cu) (net 3))
+  (segment (start 108.5 107.5) (end 108.5 108.15) (width 0.25) (layer F.Cu) (net 3))
+  (segment (start 108.5 108.15) (end 108.774999 108.424999) (width 0.25) (layer F.Cu) (net 3))
+  (segment (start 108 106) (end 108 107) (width 0.25) (layer F.Cu) (net 3))
+  (segment (start 108 107) (end 108.5 107.5) (width 0.25) (layer F.Cu) (net 3))
   (segment (start 110.25 95.5) (end 110.25 97.5) (width 0.25) (layer F.Cu) (net 3))
   (segment (start 110.25 97.5) (end 110.625 97.875) (width 0.25) (layer F.Cu) (net 3))
@@
   (segment (start 102.25 95.5) (end 105 95.5) (width 0.25) (layer B.Cu) (net 3))
   (segment (start 101.75 95) (end 102.25 95.5) (width 0.25) (layer B.Cu) (net 3))
-  (segment (start 111.5 108.5) (end 111.5 109.75) (width 0.25) (layer F.Cu) (net 3))
   (segment (start 122 97.5) (end 122 96.5) (width 0.25) (layer F.Cu) (net 3))
   (segment (start 122 96.5) (end 121.25 95.75) (width 0.25) (layer F.Cu) (net 3))
@@
   (segment (start 119.25 99.5) (end 119.25 98.75) (width 0.25) (layer F.Cu) (net 3))
   (segment (start 118.75 100) (end 119.25 99.5) (width 0.25) (layer F.Cu) (net 3))
-  (segment (start 108 106) (end 108 107.5) (width 0.25) (layer F.Cu) (net 3))
-  (segment (start 108.75 108.25) (end 111.25 108.25) (width 0.25) (layer F.Cu) (net 3))
-  (segment (start 108 107.5) (end 108.75 108.25) (width 0.25) (layer F.Cu) (net 3))
-  (segment (start 111.25 108.25) (end 111.5 108.5) (width 0.25) (layer F.Cu) (net 3))
   (segment (start 102.5 104.5) (end 102 104.5) (width 0.25) (layer F.Cu) (net 3))
   (segment (start 102 104.5) (end 101.75 104.75) (width 0.25) (layer F.Cu) (net 3))
